Commit message: makeing progress

File: urdf/head_2d.urdf (robot description, URDF)
Before this commit: robot head_2d, 2 links, 1 joints
Links:
- added link dummy
- link base_link: mass None -> 5; geometry collision box size=1 1 1; visual box size=1 1 1
- link laser: geometry visual cylinder length=0.03 radius=0.07
Joints:
- added joint dummy_joint: type fixed, parent dummy, child base_link
- joint laser_joint: origin xyz=0 0 0.05 rpy=0 0 3.1415926 -> xyz=0 0 0.51 rpy=0 0 3.1415926

Commit message: curret

File: urdf/head_2d.urdf (robot description, URDF)
Before this commit: robot head_2d, 3 links, 2 joints
Links:
- link base_link: geometry collision box size=1 1 1; visual box size=0.8 1.2 0.75
Joints:
- joint laser_joint: origin xyz=0 0 0.51 rpy=0 0 3.1415926 -> xyz=0 0 0.51 rpy=0 0 1.57075

Commit message: stand head_2d.urdf

File: urdf/head_2d.urdf (robot description, URDF)
Before this commit: robot head_2d, 3 links, 2 joints
Links:
- added link bridge_stand; visual cylinder length=0.8 radius=0.04
- added link left_stand; visual cylinder length=1.665 radius=0.04
- added link right_stand; visual cylinder length=1.665 radius=0.04
- link base_link: geometry collision box size=1 1 1; visual box size=1.2 0.8 0.75
Joints:
- added joint base_to_left_stand: type fixed, parent base_link, child left_stand, origin xyz=0 0 0.28
- added joint base_to_right_stand: type fixed, parent base_link, child right_stand, origin xyz=0 0 0.28
- added joint bridge_stand_to_left_stand: type fixed, parent left_stand, child bridge_stand, origin xyz=0 0 0
- joint laser_joint: origin xyz=0 0 0.51 rpy=0 0 1.57075 -> xyz=0 0 0.375 rpy=0 0 1.57075

Commit message: placed lazr!

File: urdf/head_2d.urdf (robot description, URDF)
Before this commit: robot mrm, 6 links, 5 joints
Joints:
- joint base_to_left_stand: origin xyz=0 0 0.28 -> xyz=-0.2 0.4 0.28
- joint base_to_right_stand: origin xyz=0 0 0.28 -> xyz=-0.2 -0.4 0.28
- joint bridge_stand_to_left_stand: origin xyz=0 0 0 -> xyz=0 -0.4 1.665
- joint laser_joint: origin xyz=0 0 0.375 rpy=0 0 1.57075 -> xyz=0 0 0.04 rpy=0 0 1.57075; parent base_link -> bridge_stand

Commit message: add camera_link

File: urdf/head_2d.urdf (robot description, URDF)
Before this commit: robot mrm, 6 links, 5 joints
Links:
- added link camera_link; visual box size=0.05 0.05 0.05
Joints:
- added joint camera_joint: type fixed, parent bridge_stand, child camera_link, origin xyz=0.047 0.0 0.0 rpy=0 0 0, axis 1 0 0

Commit message: camera orientation head_2d.urdf

File: urdf/head_2d.urdf (robot description, URDF)
Before this commit: robot mrm, 7 links, 6 joints
Joints:
- joint camera_joint: axis 1 0 0 -> 0 0 0; origin xyz=0.047 0.0 0.0 rpy=0 0 0 -> xyz=0.047 0.0 0.0 rpy=0 2.740164 3.14159
- joint laser_joint: origin xyz=0 0 0.04 rpy=0 0 1.57075 -> xyz=0 0 0.04 rpy=0 0 3.14159
